File: Boards/AnalogInputV1-1/Analog-Input-Card.sch (KiCad schematic (older format))
At the start: 18 parts, among them IC1 PIC16F1783, J1 5Vdc Jumper, P1 AquaPicBus, P2 Inputs, P3 ICSP, P4 Power, P5 EARTH GROUND, Q1 AO3407A, U1 ST485EC, X1 8MHz

Commit message: started ananlog input revision 2
Parts:
- added C?: 100nF, Capacitors_SMD:C_0805, symbol C-RESCUE-Analog-Input-Card
- added U?: MCP3428, symbol MCP3428
Connections:
- net +5V: now also U?.6 (VDD)
- net GND: now also U?.12 (CH3-), U?.14 (CH4-), U?.2 (CH1-), U?.4 (CH2-), U?.5 (VSS)
- net Input1: now also U?.1 (CH1+); no longer IC1.2 (RA0)
- net Input2: now also U?.3 (CH2+); no longer IC1.3 (RA1)
- net Input3: now also U?.11 (CH3+); no longer IC1.4 (RA2)
- net Input4: now also U?.13 (CH4+); no longer IC1.5 (RA3)
- no-connect marks 11 -> 15
Other:
- moved on the sheet: C2, P1, P2, U1
