File: Boards/AnalogInputV2-0/Analog-Input-Card.sch (KiCad schematic (older format))
At the start: 34 parts, among them IC1 PIC16F18855, J1 5Vdc Jumper, P1 AquaPicBus, P2 Inputs, P3 EARTH GROUND, P4 Power, P5 ICSP, Q1 AO3407A, U1 ST485EC, U2 MCP3428, X1 8MHz

Commit message: documentation for rev 2 analog input
Parts:
- R10, R11, R12, R13, R14, R7, R8, R9: footprint (none) -> Resistors_SMD:R_0805; Comment (none) -> 0805, 1/4W, 1%, Thin Film
- R5, R6: footprint (none) -> Resistors_SMD:R_0805
- RV1, RV2, RV3, RV4: footprint (none) -> A_MyFootPrints:POTENTIAMETER_SMD
Changed lines of the file:
@@
 F 0 "R7" V 8130 900 50  0000 C CNN
 F 1 "4K32" V 8050 900 50  0000 C CNN
-F 2 "" V 7980 900 50  0001 C CNN
+F 2 "Resistors_SMD:R_0805" V 7980 900 50  0001 C CNN
 F 3 "" H 8050 900 50  0001 C CNN
+F 4 "0805, 1/4W, 1%, Thin Film" V 8050 900 60  0001 C CNN "Comment"
 	1    8050 900
 	0    1    1    0
@@
 F 0 "R8" V 8530 900 50  0000 C CNN
 F 1 "10K" V 8450 900 50  0000 C CNN
-F 2 "" V 8380 900 50  0001 C CNN
+F 2 "Resistors_SMD:R_0805" V 8380 900 50  0001 C CNN
 F 3 "" H 8450 900 50  0001 C CNN
+F 4 "0805, 1/4W, 1%, Thin Film" V 8450 900 60  0001 C CNN "Comment"
 	1    8450 900
 	0    1    1    0
@@
 F 0 "RV1" V 7625 1150 50  0000 C CNN
 F 1 "10K" V 7700 1150 50  0000 C CNN
-F 2 "" H 7800 1150 50  0001 C CNN
+F 2 "A_MyFootPrints:POTENTIAMETER_SMD" H 7800 1150 50  0001 C CNN
 F 3 "" H 7800 1150 50  0001 C CNN
 	1    7800 1150
@@
 F 0 "R9" V 8130 1700 50  0000 C CNN
 F 1 "4K32" V 8050 1700 50  0000 C CNN
-F 2 "" V 7980 1700 50  0001 C CNN
+F 2 "Resistors_SMD:R_0805" V 7980 1700 50  0001 C CNN
 F 3 "" H 8050 1700 50  0001 C CNN
+F 4 "0805, 1/4W, 1%, Thin Film" V 8050 1700 60  0001 C CNN "Comment"
 	1    8050 1700
 	0    1    1    0
@@
 F 0 "R10" V 8530 1700 50  0000 C CNN
 F 1 "10K" V 8450 1700 50  0000 C CNN
-F 2 "" V 8380 1700 50  0001 C CNN
+F 2 "Resistors_SMD:R_0805" V 8380 1700 50  0001 C CNN
 F 3 "" H 8450 1700 50  0001 C CNN
+F 4 "0805, 1/4W, 1%, Thin Film" V 8450 1700 60  0001 C CNN "Comment"
 	1    8450 1700
 	0    1    1    0
@@
 F 0 "RV2" V 7625 1950 50  0000 C CNN
 F 1 "10K" V 7700 1950 50  0000 C CNN
-F 2 "" H 7800 1950 50  0001 C CNN
+F 2 "A_MyFootPrints:POTENTIAMETER_SMD" H 7800 1950 50  0001 C CNN
 F 3 "" H 7800 1950 50  0001 C CNN
 	1    7800 1950
@@
 F 0 "R11" V 8130 2500 50  0000 C CNN
 F 1 "4K32" V 8050 2500 50  0000 C CNN
-F 2 "" V 7980 2500 50  0001 C CNN
+F 2 "Resistors_SMD:R_0805" V 7980 2500 50  0001 C CNN
 F 3 "" H 8050 2500 50  0001 C CNN
+F 4 "0805, 1/4W, 1%, Thin Film" V 8050 2500 60  0001 C CNN "Comment"
 	1    8050 2500
 	0    1    1    0
@@
 F 0 "R12" V 8530 2500 50  0000 C CNN
 F 1 "10K" V 8450 2500 50  0000 C CNN
-F 2 "" V 8380 2500 50  0001 C CNN
+F 2 "Resistors_SMD:R_0805" V 8380 2500 50  0001 C CNN
 F 3 "" H 8450 2500 50  0001 C CNN
+F 4 "0805, 1/4W, 1%, Thin Film" V 8450 2500 60  0001 C CNN "Comment"
 	1    8450 2500
 	0    1    1    0
@@
 F 0 "RV3" V 7625 2750 50  0000 C CNN
 F 1 "10K" V 7700 2750 50  0000 C CNN
-F 2 "" H 7800 2750 50  0001 C CNN
+F 2 "A_MyFootPrints:POTENTIAMETER_SMD" H 7800 2750 50  0001 C CNN
 F 3 "" H 7800 2750 50  0001 C CNN
 	1    7800 2750
@@
 F 0 "R13" V 8130 3300 50  0000 C CNN
 F 1 "4K32" V 8050 3300 50  0000 C CNN
-F 2 "" V 7980 3300 50  0001 C CNN
+F 2 "Resistors_SMD:R_0805" V 7980 3300 50  0001 C CNN
 F 3 "" H 8050 3300 50  0001 C CNN
+F 4 "0805, 1/4W, 1%, Thin Film" V 8050 3300 60  0001 C CNN "Comment"
 	1    8050 3300
 	0    1    1    0
@@
 F 0 "R14" V 8530 3300 50  0000 C CNN
 F 1 "10K" V 8450 3300 50  0000 C CNN
-F 2 "" V 8380 3300 50  0001 C CNN
+F 2 "Resistors_SMD:R_0805" V 8380 3300 50  0001 C CNN
 F 3 "" H 8450 3300 50  0001 C CNN
+F 4 "0805, 1/4W, 1%, Thin Film" V 8450 3300 60  0001 C CNN "Comment"
 	1    8450 3300
 	0    1    1    0
@@
 F 0 "RV4" V 7625 3550 50  0000 C CNN
 F 1 "10K" V 7700 3550 50  0000 C CNN
-F 2 "" H 7800 3550 50  0001 C CNN
+F 2 "A_MyFootPrints:POTENTIAMETER_SMD" H 7800 3550 50  0001 C CNN
 F 3 "" H 7800 3550 50  0001 C CNN
 	1    7800 3550
@@
 F 0 "R5" V 3780 2550 50  0000 C CNN
 F 1 "4K7" V 3700 2550 50  0000 C CNN
-F 2 "" V 3630 2550 50  0001 C CNN
+F 2 "Resistors_SMD:R_0805" V 3630 2550 50  0001 C CNN
 F 3 "" H 3700 2550 50  0001 C CNN
 	1    3700 2550
@@
 F 0 "R6" V 3980 2550 50  0000 C CNN
 F 1 "4K7" V 3900 2550 50  0000 C CNN
-F 2 "" V 3830 2550 50  0001 C CNN
+F 2 "Resistors_SMD:R_0805" V 3830 2550 50  0001 C CNN
 F 3 "" H 3900 2550 50  0001 C CNN
 	1    3900 2550

Commit message: work on ai v2
Parts:
- IC1: footprint (none) -> Housings_DFN_QFN:QFN-28-1EP_6x6mm_Pitch0.65mm
- P3: value EARTH GROUND -> Earth
- R5, R6: value 4K7 -> 4K32
- U2: footprint (none) -> Housings_SSOP:TSSOP-14_4.4x5mm_Pitch0.65mm
Changed lines of the file:
@@
 P 10200 3500
 F 0 "P3" H 10200 3600 50  0000 C CNN
-F 1 "EARTH GROUND" V 10300 3500 50  0000 C CNN
+F 1 "Earth" V 10300 3500 50  0000 C CNN
 F 2 "Pin_Headers:Pin_Header_Straight_1x01" H 10200 3500 60  0001 C CNN
 F 3 "" H 10200 3500 60  0000 C CNN
@@
 F 0 "U2" H 5550 2550 50  0000 R CNN
 F 1 "MCP3428" H 5800 2550 50  0000 L CNN
-F 2 "" H 5700 2100 50  0001 C CNN
+F 2 "Housings_SSOP:TSSOP-14_4.4x5mm_Pitch0.65mm" H 5700 2100 50  0001 C CNN
 F 3 "" H 5700 2100 50  0001 C CNN
 	1    5700 2100
@@
 F 0 "IC1" H 2250 3300 60  0000 C CNN
 F 1 "PIC16F18855" H 2700 900 60  0000 C CNN
-F 2 "" H 2700 2100 60  0000 C CNN
+F 2 "Housings_DFN_QFN:QFN-28-1EP_6x6mm_Pitch0.65mm" H 2700 2100 60  0001 C CNN
 F 3 "" H 2700 2100 60  0000 C CNN
 	1    2600 2100
@@
 P 3700 2550
 F 0 "R5" V 3780 2550 50  0000 C CNN
-F 1 "4K7" V 3700 2550 50  0000 C CNN
+F 1 "4K32" V 3700 2550 50  0000 C CNN
 F 2 "Resistors_SMD:R_0805" V 3630 2550 50  0001 C CNN
 F 3 "" H 3700 2550 50  0001 C CNN
@@
 P 3900 2550
 F 0 "R6" V 3980 2550 50  0000 C CNN
-F 1 "4K7" V 3900 2550 50  0000 C CNN
+F 1 "4K32" V 3900 2550 50  0000 C CNN
 F 2 "Resistors_SMD:R_0805" V 3830 2550 50  0001 C CNN
 F 3 "" H 3900 2550 50  0001 C CNN

Commit message: worked on i2c driver and board design
Parts:
- removed J1: 5Vdc Jumper, Pin_Headers:Pin_Header_Straight_1x03, symbol CONN_01X03
- added C4, C5, C6, C7: 100nF, Capacitors_SMD:C_0805, symbol C_Small
- added D10, D4, D6, D8: SMBJ30D, Diodes_SMD:D_SMB, symbol D_TVS_ALT
- added D3, D5, D7, D9: BZX84C4V7, Diodes_SMD:D_SOT-23_ANK, symbol D_Zener_ALT
- D1: footprint A_MyFootPrints:PLCC-4 -> MyFootPrints:PLCC-4
- IC1: footprint Housings_DFN_QFN:QFN-28-1EP_6x6mm_Pitch0.65mm -> Housings_SSOP:SSOP-28_5.3x10.2mm_Pitch0.65mm
- P1: footprint A_MyFootPrints:USB-1.1_Stacked -> MyFootPrints:USB-1.1_Stacked
- P2: footprint A_MyFootPrints:Screw_Header_1x16 -> MyFootPrints:Screw_Header_1x16
- P3: footprint Pin_Headers:Pin_Header_Straight_1x01 -> MyFootPrints:Screw_Header_1x2; symbol CONN_01X01 -> CONN_01X02
- P4: footprint A_MyFootPrints:Screw_Header_1x2 -> MyFootPrints:Screw_Header_1x2
- P5: footprint Pin_Headers:Pin_Header_Straight_1x06 -> Pin_Headers:Pin_Header_Straight_1x06_Pitch2.54mm
- RV1, RV2, RV3, RV4: footprint A_MyFootPrints:POTENTIAMETER_SMD -> MyFootPrints:POTENTIAMETER_SMD
- X1: footprint A_MyFootPrints:Resonator_3.2x1.3 -> MyFootPrints:Resonator_3.2x1.3
Connections:
- net labels removed: 5Vdc, 5VdcA, 5VdcB, GNDPWR
- wire segments 127 -> 136
Other:
- note added: "Input Protection and Voltage Dividers"
- note added: "Power Input and Reverse Cicuit Protection"
- note removed: "+5Vdc Jumper"
- note removed: "Input Voltage Dividers"
- note removed: "Power Connector"
- note removed: "Reverse Cicuit Protection"
- moved on the sheet: C1, C2, C3, D1, D2, IC1, P1, P2, P4, P5, Q1, R1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

Commit message: started development with PIC32MM
Parts:
- removed C1: 100nF, Capacitors_SMD:C_0805, symbol C-RESCUE-Analog-Input-Card
- removed IC1: PIC16F18855, Housings_SSOP:SSOP-28_5.3x10.2mm_Pitch0.65mm, symbol PIC16F18855
- added C1, C8: 100nF, Capacitors_SMD:C_0805, symbol C_Small
- added C10, C9: 4u7, Capacitors_SMD:C_0805, symbol C_Small
- added IC1: PIC32MM0064GPM028, Housings_DFN_QFN:QFN-28-1EP_6x6mm_Pitch0.65mm, symbol PIC32MM0064GPM028_QFN
- added Q2, Q3, Q4: NX7002AK, Housings_SOT-23_SOT-143_TSOT-6:SOT-23, symbol MOSFET_N_SMALL
- added R15, R16, R17, R18: 4K32, Resistors_SMD:R_0805, symbol R
- added R19: 1K, Resistors_SMD:R_0805, symbol R
- added R20, R21: 10K, Resistors_SMD:R_0805, symbol R
- added U3: AP2114H, TO_SOT_Packages_SMD:SOT-223, symbol AP1117-33
- D3, D5, D7, D9: value BZX84C4V7 -> BZX84C3V3
- R1, R2: symbol R-RESCUE-Analog-Input-Card -> R
- R3: renamed from R4; symbol R-RESCUE-Analog-Input-Card -> R
- R7, R9: value 4K32 -> 4K99
- renumbered R3 to R4
Connections:
- net +5V: now also C9.1, R16.1, R18.1, R21.1, U3.3 (VI); no longer C3.1, D1.4, P5.2 (P2), R5.1, R6.1, U2.6 (VDD)
- net /MCLR: now also IC1.26 (/MCLR)
- net Ch1: now also R7.2, R8.2; no longer RV1.2
- net Ch2: now also R10.2, R9.2; no longer RV2.2
- net Ch3: now also R11.2, R12.2; no longer RV3.2
- net Ch4: now also R13.2, R14.2; no longer RV4.2
- net GND: now also R10.1, R12.1, R14.1, R8.1, X1.2 (G), C1.2, C10.2, C8.2, C9.2, IC1.24 (AVss), IC1.5 (Vss), Q4.2 (S), R20.2, U3.1 (GND); no longer RV1.1, RV2.1, RV3.1, RV4.1
- net Input1: now also RV1.1; no longer R8.1
- net Input2: now also RV2.1; no longer R10.1
- net Input3: now also RV3.1; no longer R12.1
- net Input4: now also RV4.1; no longer R14.1
- net PGC: now also IC1.27 (RA0)
- net PGD: now also IC1.28 (RA1)
- net RX: now also Q3.3 (D), R18.2
- net SCL: now also IC1.16 (RC9)
- net SDA: now also IC1.11 (RB5)
- net TX: now also Q2.3 (D), R16.2
- net at X1.1 (X2): now also IC1.7 (RA3/OSC2)
- net at X1.3 (X1): now also IC1.6 (RA2/OSC1)
- net at R7.1: now also RV1.2, RV1.3; no longer R8.2
- net at R9.1: now also RV2.2, RV2.3; no longer R10.2
- net at R11.1: now also RV3.2, RV3.3; no longer R12.2
- net at R13.1: now also RV4.2, RV4.3; no longer R14.2
- net D+ renamed A
- net D- renamed B
- net STAT_LED_G renamed LED_G
- net LED_G: now also IC1.2 (RB1)
- net STAT_LED_R renamed LED_R
- net LED_R: now also IC1.1 (RB0)
- net STAT_LED_Y renamed LED_Y
- net LED_Y: now also IC1.3 (RB2)
- net T_nR renamed RTS
- net RTS: now also Q4.3 (D), R21.2
- new net: C8.1, IC1.17 (Vcap)
- new net: Q4.1 (G), R19.1, R20.1
- new net +3V3: C1.1, C10.1, C3.1, D1.4, IC1.10 (Vdd), IC1.25 (AVdd), P5.2 (P2), Q2.1 (G), Q3.1 (G), R15.1, R17.1, R5.1, R6.1, U2.6 (VDD), U3.2 (VO)
- new net /RTS: IC1.14 (RB8), IC1.15 (RB9), R19.2
- new net RX_LV: IC1.23 (RB15), Q3.2 (S), R17.2
- new net TX_LV: IC1.22 (RB14), Q2.2 (S), R15.2
- no-connect marks 13 -> 10
Other:
- note added: "3.3V LDO"
- note added: "Level Shift"
- note added: "NOT and Level Shift"
- note added: "With an input of 5V:\nThe output will be 3.336V with RVx at 0R\nThe output will be 2.001V with RVx at 10K\nVout = (Vin * 10) / (24.99 - RVx)"
- moved on the sheet: C2, C4, C5, C6, C7, D1, D10, D2, D3, D4, D5, D6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

Commit message: finished board layout for ai
Parts:
- IC1: footprint Housings_DFN_QFN:QFN-28-1EP_6x6mm_Pitch0.65mm -> Housings_SSOP:SSOP-28_5.3x10.2mm_Pitch0.65mm
- Q1, Q2, Q3, Q4: footprint Housings_SOT-23_SOT-143_TSOT-6:SOT-23 -> TO_SOT_Packages_SMD:SOT-23
- R11, R13, R15, R16, R17, R18, R5, R6: value 4K32 -> 4K99
Changed lines of the file:
@@
 F 0 "Q1" V 10150 5750 60  0000 R CNN
 F 1 "AO3407A" V 9750 5500 60  0000 R CNN
-F 2 "Housings_SOT-23_SOT-143_TSOT-6:SOT-23" H 9900 5600 60  0001 C CNN
+F 2 "TO_SOT_Packages_SMD:SOT-23" H 9900 5600 60  0001 C CNN
 F 3 "" H 9900 5600 60  0000 C CNN
 	1    9900 5600
@@
 P 8250 3100
 F 0 "R11" V 8330 3100 50  0000 C CNN
-F 1 "4K32" V 8250 3100 50  0000 C CNN
+F 1 "4K99" V 8250 3100 50  0000 C CNN
 F 2 "Resistors_SMD:R_0805" V 8180 3100 50  0001 C CNN
 F 3 "" H 8250 3100 50  0001 C CNN
@@
 P 8250 3900
 F 0 "R13" V 8330 3900 50  0000 C CNN
-F 1 "4K32" V 8250 3900 50  0000 C CNN
+F 1 "4K99" V 8250 3900 50  0000 C CNN
 F 2 "Resistors_SMD:R_0805" V 8180 3900 50  0001 C CNN
 F 3 "" H 8250 3900 50  0001 C CNN
@@
 P 3300 3050
 F 0 "R5" V 3380 3050 50  0000 C CNN
-F 1 "4K32" V 3300 3050 50  0000 C CNN
+F 1 "4K99" V 3300 3050 50  0000 C CNN
 F 2 "Resistors_SMD:R_0805" V 3230 3050 50  0001 C CNN
 F 3 "" H 3300 3050 50  0001 C CNN
@@
 P 3300 1750
 F 0 "R6" V 3380 1750 50  0000 C CNN
-F 1 "4K32" V 3300 1750 50  0000 C CNN
+F 1 "4K99" V 3300 1750 50  0000 C CNN
 F 2 "Resistors_SMD:R_0805" V 3230 1750 50  0001 C CNN
 F 3 "" H 3300 1750 50  0001 C CNN
@@
 F 0 "IC1" H 1800 3350 60  0000 C CNN
 F 1 "PIC32MM0064GPM028" H 2100 850 60  0000 C CNN
-F 2 "Housings_DFN_QFN:QFN-28-1EP_6x6mm_Pitch0.65mm" H 2400 1650 60  0001 C CNN
+F 2 "Housings_SSOP:SSOP-28_5.3x10.2mm_Pitch0.65mm" H 2400 1650 60  0001 C CNN
 F 3 "" H 2400 1650 60  0001 C CNN
 	1    2100 2100
@@
 F 0 "Q3" V 3000 5200 60  0000 R CNN
 F 1 "NX7002AK" V 3350 5250 60  0000 R CNN
-F 2 "Housings_SOT-23_SOT-143_TSOT-6:SOT-23" H 3100 5100 60  0001 C CNN
+F 2 "TO_SOT_Packages_SMD:SOT-23" H 3100 5100 60  0001 C CNN
 F 3 "" H 3100 5100 60  0000 C CNN
 	1    3100 5100
@@
 P 2800 5050
 F 0 "R17" V 2880 5050 50  0000 C CNN
-F 1 "4K32" V 2807 5051 50  0000 C CNN
+F 1 "4K99" V 2807 5051 50  0000 C CNN
 F 2 "Resistors_SMD:R_0805" V 2730 5050 30  0001 C CNN
 F 3 "" H 2800 5050 30  0000 C CNN
@@
 P 3400 5050
 F 0 "R18" V 3480 5050 50  0000 C CNN
-F 1 "4K32" V 3407 5051 50  0000 C CNN
+F 1 "4K99" V 3407 5051 50  0000 C CNN
 F 2 "Resistors_SMD:R_0805" V 3330 5050 30  0001 C CNN
 F 3 "" H 3400 5050 30  0000 C CNN
@@
 F 0 "Q4" H 1800 5000 60  0000 R CNN
 F 1 "NX7002AK" V 2050 4950 60  0000 R CNN
-F 2 "Housings_SOT-23_SOT-143_TSOT-6:SOT-23" H 1800 4800 60  0001 C CNN
+F 2 "TO_SOT_Packages_SMD:SOT-23" H 1800 4800 60  0001 C CNN
 F 3 "" H 1800 4800 60  0000 C CNN
 	1    1800 4800
@@
 F 0 "Q2" V 3000 4400 60  0000 R CNN
 F 1 "NX7002AK" V 3350 4450 60  0000 R CNN
-F 2 "Housings_SOT-23_SOT-143_TSOT-6:SOT-23" H 3100 4300 60  0001 C CNN
+F 2 "TO_SOT_Packages_SMD:SOT-23" H 3100 4300 60  0001 C CNN
 F 3 "" H 3100 4300 60  0000 C CNN
 	1    3100 4300
@@
 P 2800 4250
 F 0 "R15" V 2880 4250 50  0000 C CNN
-F 1 "4K32" V 2807 4251 50  0000 C CNN
+F 1 "4K99" V 2807 4251 50  0000 C CNN
 F 2 "Resistors_SMD:R_0805" V 2730 4250 30  0001 C CNN
 F 3 "" H 2800 4250 30  0000 C CNN
@@
 P 3400 4250
 F 0 "R16" V 3480 4250 50  0000 C CNN
-F 1 "4K32" V 3407 4251 50  0000 C CNN
+F 1 "4K99" V 3407 4251 50  0000 C CNN
 F 2 "Resistors_SMD:R_0805" V 3330 4250 30  0001 C CNN
 F 3 "" H 3400 4250 30  0000 C CNN

Commit message: cleaning up a few things
Other:
- note added: "With an input of 5V:\nThe output will be 3.336V with RVx at 10K\nThe output will be 2.001V with RVx at 0R, bypassed\nVout = (Vin * 10) / (14.99 + RVx)"
- note removed: "With an input of 5V:\nThe output will be 3.336V with RVx at 0R\nThe output will be 2.001V with RVx at 10K\nVout = (Vin * 10) / (24.99 - RVx)"
- moved on the sheet: Q2, Q3, R15, R16, R17, R18
Changed lines of the file:
@@
 NoConn ~ 2700 2600
 NoConn ~ 2700 2700
-Text Label 3700 4400 2    60   ~ 0
+Text Label 3800 4400 2    60   ~ 0
 TX
-Text Label 2400 4400 0    60   ~ 0
+Text Label 2500 4400 0    60   ~ 0
 TX_LV
 Text Label 3100 2800 2    60   ~ 0
@@
 L MOSFET_N_SMALL Q3
 U 1 1 5A099F7B
-P 3100 5100
-F 0 "Q3" V 3000 5200 60  0000 R CNN
-F 1 "NX7002AK" V 3350 5250 60  0000 R CNN
-F 2 "TO_SOT_Packages_SMD:SOT-23" H 3100 5100 60  0001 C CNN
-F 3 "" H 3100 5100 60  0000 C CNN
-	1    3100 5100
+P 3200 5100
+F 0 "Q3" V 3100 5200 60  0000 R CNN
+F 1 "NX7002AK" V 3450 5250 60  0000 R CNN
+F 2 "TO_SOT_Packages_SMD:SOT-23" H 3200 5100 60  0001 C CNN
+F 3 "" H 3200 5100 60  0000 C CNN
+	1    3200 5100
 	0    1    1    0
 $EndComp
-Text Label 3700 5200 2    60   ~ 0
+Text Label 3800 5200 2    60   ~ 0
 RX
-Text Label 2400 5200 0    60   ~ 0
+Text Label 2500 5200 0    60   ~ 0
 RX_LV
 $Comp
 L R R17
 U 1 1 5A099F8F
-P 2800 5050
-F 0 "R17" V 2880 5050 50  0000 C CNN
-F 1 "4K99" V 2807 5051 50  0000 C CNN
-F 2 "Resistors_SMD:R_0805" V 2730 5050 30  0001 C CNN
-F 3 "" H 2800 5050 30  0000 C CNN
-	1    2800 5050
+P 2900 5050
+F 0 "R17" V 2980 5050 50  0000 C CNN
+F 1 "4K99" V 2907 5051 50  0000 C CNN
+F 2 "Resistors_SMD:R_0805" V 2830 5050 30  0001 C CNN
+F 3 "" H 2900 5050 30  0000 C CNN
+	1    2900 5050
 	1    0    0    -1
 $EndComp
@@
 L R R18
 U 1 1 5A099F95
-P 3400 5050
-F 0 "R18" V 3480 5050 50  0000 C CNN
-F 1 "4K99" V 3407 5051 50  0000 C CNN
-F 2 "Resistors_SMD:R_0805" V 3330 5050 30  0001 C CNN
-F 3 "" H 3400 5050 30  0000 C CNN
-	1    3400 5050
+P 3500 5050
+F 0 "R18" V 3580 5050 50  0000 C CNN
+F 1 "4K99" V 3507 5051 50  0000 C CNN
+F 2 "Resistors_SMD:R_0805" V 3430 5050 30  0001 C CNN
+F 3 "" H 3500 5050 30  0000 C CNN
+	1    3500 5050
 	1    0    0    -1
 $EndComp
@@
 L +5V #PWR042
 U 1 1 5A0A9815
-P 3400 4800
-F 0 "#PWR042" H 3400 4890 20  0001 C CNN
-F 1 "+5V" H 3400 4890 30  0000 C CNN
-F 2 "~" H 3400 4800 60  0000 C CNN
-F 3 "~" H 3400 4800 60  0000 C CNN
-	1    3400 4800
+P 3500 4800
+F 0 "#PWR042" H 3500 4890 20  0001 C CNN
+F 1 "+5V" H 3500 4890 30  0000 C CNN
+F 2 "~" H 3500 4800 60  0000 C CNN
+F 3 "~" H 3500 4800 60  0000 C CNN
+	1    3500 4800
 	1    0    0    -1
 $EndComp
@@
 L +3.3V #PWR043
 U 1 1 5A0AB287
-P 2800 4800
-F 0 "#PWR043" H 2800 4650 50  0001 C CNN
-F 1 "+3.3V" H 2800 4900 30  0000 C CNN
-F 2 "" H 2800 4800 50  0001 C CNN
-F 3 "" H 2800 4800 50  0001 C CNN
-	1    2800 4800
+P 2900 4800
+F 0 "#PWR043" H 2900 4650 50  0001 C CNN
+F 1 "+3.3V" H 2900 4900 30  0000 C CNN
+F 2 "" H 2900 4800 50  0001 C CNN
+F 3 "" H 2900 4800 50  0001 C CNN
+	1    2900 4800
 	1    0    0    -1
 $EndComp
@@
 $EndComp
 Text Notes 6900 1200 0    60   ~ 0
-With an input of 5V:\nThe output will be 3.336V with RVx at 0R\nThe output will be 2.001V with RVx at 10K\nVout = (Vin * 10) / (24.99 - RVx)
+With an input of 5V:\nThe output will be 3.336V with RVx at 10K\nThe output will be 2.001V with RVx at 0R, bypassed\nVout = (Vin * 10) / (14.99 + RVx)
 Wire Wire Line
 	5150 2950 5750 2950
@@
 Connection ~ 2800 2300
 Wire Wire Line
-	2400 5200 2900 5200
-Connection ~ 2800 5200
+	2500 5200 3000 5200
+Connection ~ 2900 5200
 Wire Wire Line
 	1900 4400 1900 4600
@@
 	7200 3500 7200 3450
 Wire Wire Line
-	3400 4800 3400 4900
-Wire Wire Line
-	2800 4800 2800 4900
-Wire Wire Line
-	2800 4850 3000 4850
-Wire Wire Line
-	3000 4850 3000 4900
-Connection ~ 2800 4850
-Wire Wire Line
-	3300 5200 3700 5200
-Connection ~ 3400 5200
+	3500 4800 3500 4900
+Wire Wire Line
+	2900 4800 2900 4900
+Wire Wire Line
+	2900 4850 3100 4850
+Wire Wire Line
+	3100 4850 3100 4900
+Connection ~ 2900 4850
+Wire Wire Line
+	3400 5200 3800 5200
+Connection ~ 3500 5200
 $Comp
 L MOSFET_N_SMALL Q2
 U 1 1 5A0D44E8
-P 3100 4300
-F 0 "Q2" V 3000 4400 60  0000 R CNN
-F 1 "NX7002AK" V 3350 4450 60  0000 R CNN
-F 2 "TO_SOT_Packages_SMD:SOT-23" H 3100 4300 60  0001 C CNN
-F 3 "" H 3100 4300 60  0000 C CNN
-	1    3100 4300
+P 3200 4300
+F 0 "Q2" V 3100 4400 60  0000 R CNN
+F 1 "NX7002AK" V 3450 4450 60  0000 R CNN
+F 2 "TO_SOT_Packages_SMD:SOT-23" H 3200 4300 60  0001 C CNN
+F 3 "" H 3200 4300 60  0000 C CNN
+	1    3200 4300
 	0    1    1    0
 $EndComp
@@
 L R R15
 U 1 1 5A0D44F0
-P 2800 4250
-F 0 "R15" V 2880 4250 50  0000 C CNN
-F 1 "4K99" V 2807 4251 50  0000 C CNN
-F 2 "Resistors_SMD:R_0805" V 2730 4250 30  0001 C CNN
-F 3 "" H 2800 4250 30  0000 C CNN
-	1    2800 4250
+P 2900 4250
+F 0 "R15" V 2980 4250 50  0000 C CNN
+F 1 "4K99" V 2907 4251 50  0000 C CNN
+F 2 "Resistors_SMD:R_0805" V 2830 4250 30  0001 C CNN
+F 3 "" H 2900 4250 30  0000 C CNN
+	1    2900 4250
 	1    0    0    -1
 $EndComp
@@
 L R R16
 U 1 1 5A0D44F6
-P 3400 4250
-F 0 "R16" V 3480 4250 50  0000 C CNN
-F 1 "4K99" V 3407 4251 50  0000 C CNN
-F 2 "Resistors_SMD:R_0805" V 3330 4250 30  0001 C CNN
-F 3 "" H 3400 4250 30  0000 C CNN
-	1    3400 4250
+P 3500 4250
+F 0 "R16" V 3580 4250 50  0000 C CNN
+F 1 "4K99" V 3507 4251 50  0000 C CNN
+F 2 "Resistors_SMD:R_0805" V 3430 4250 30  0001 C CNN
+F 3 "" H 3500 4250 30  0000 C CNN
+	1    3500 4250
 	1    0    0    -1
 $EndComp
@@
 L +5V #PWR051
 U 1 1 5A0D44FC
-P 3400 4000
-F 0 "#PWR051" H 3400 4090 20  0001 C CNN
-F 1 "+5V" H 3400 4090 30  0000 C CNN
-F 2 "~" H 3400 4000 60  0000 C CNN
-F 3 "~" H 3400 4000 60  0000 C CNN
-	1    3400 4000
+P 3500 4000
+F 0 "#PWR051" H 3500 4090 20  0001 C CNN
+F 1 "+5V" H 3500 4090 30  0000 C CNN
+F 2 "~" H 3500 4000 60  0000 C CNN
+F 3 "~" H 3500 4000 60  0000 C CNN
+	1    3500 4000
 	1    0    0    -1
 $EndComp
@@
 L +3.3V #PWR052
 U 1 1 5A0D4502
-P 2800 4000
-F 0 "#PWR052" H 2800 3850 50  0001 C CNN
-F 1 "+3.3V" H 2800 4100 30  0000 C CNN
-F 2 "" H 2800 4000 50  0001 C CNN
-F 3 "" H 2800 4000 50  0001 C CNN
-	1    2800 4000
-	1    0    0    -1
-$EndComp
-Wire Wire Line
-	2400 4400 2900 4400
-Connection ~ 2800 4400
-Wire Wire Line
-	3400 4000 3400 4100
-Wire Wire Line
-	2800 4000 2800 4100
-Wire Wire Line
-	2800 4050 3000 4050
-Wire Wire Line
-	3000 4050 3000 4100
-Connection ~ 2800 4050
-Wire Wire Line
-	3300 4400 3700 4400
-Connection ~ 3400 4400
+P 2900 4000
+F 0 "#PWR052" H 2900 3850 50  0001 C CNN
+F 1 "+3.3V" H 2900 4100 30  0000 C CNN
+F 2 "" H 2900 4000 50  0001 C CNN
+F 3 "" H 2900 4000 50  0001 C CNN
+	1    2900 4000
+	1    0    0    -1
+$EndComp
+Wire Wire Line
+	2500 4400 3000 4400
+Connection ~ 2900 4400
+Wire Wire Line
+	3500 4000 3500 4100
+Wire Wire Line
+	2900 4000 2900 4100
+Wire Wire Line
+	2900 4050 3100 4050
+Wire Wire Line
+	3100 4050 3100 4100
+Connection ~ 2900 4050
+Wire Wire Line
+	3400 4400 3800 4400
+Connection ~ 3500 4400
 $Comp
 L +5V #PWR053

Commit message: fixed pinout on analog input card
Parts:
- removed D2: APT2012, LEDs:LED-0805, symbol LED-RESCUE-Analog-Input-Card
- removed R4: 300R, Resistors_SMD:R_0805, symbol R-RESCUE-Analog-Input-Card
- added C11: 100nF, Capacitors_SMD:C_0805, symbol C_Small
- added D2: APT2012, LEDs:LED-0805, symbol LED_ALT
- added R4: 150R, Resistors_SMD:R_0805, symbol R
- D1: value SMP4-RGY -> SMTL4-RGY
- IC1: symbol PIC32MM0064GPM028_QFN -> PIC32MM0064GPM028_SSOP
- R1, R2, R3: value 300R -> 150R
Connections:
- net +3V3: now also IC1.13 (Vdd), IC1.28 (AVdd), C11.1, R4.1; no longer IC1.10 (Vdd), IC1.25 (AVdd)
- net /MCLR: now also IC1.1 (/MCLR); no longer IC1.26 (/MCLR)
- net /RTS: now also IC1.17 (RB8), IC1.18 (RB9); no longer IC1.14 (RB8), IC1.15 (RB9)
- net GND: now also IC1.23 (Vusb), IC1.27 (AVss), IC1.8 (Vss), C11.2, D2.1 (K); no longer IC1.24 (AVss), IC1.5 (Vss)
- net LED_G: now also IC1.5 (RB1); no longer IC1.2 (RB1)
- net LED_R: now also IC1.4 (RB0); no longer IC1.1 (RB0)
- net LED_Y: now also IC1.6 (RB2); no longer IC1.3 (RB2)
- net PGC: now also IC1.2 (RA0); no longer IC1.27 (RA0)
- net PGD: now also IC1.3 (RA1); no longer IC1.28 (RA1)
- net RX_LV: now also IC1.26 (RB15); no longer IC1.23 (RB15)
- net SCL: now also IC1.19 (RC9); no longer IC1.16 (RC9)
- net SDA: now also IC1.14 (RB5); no longer IC1.11 (RB5)
- net TX_LV: now also IC1.25 (RB14); no longer IC1.22 (RB14)
- net at X1.1 (X2): now also IC1.10 (RA3/OSC2); no longer IC1.7 (RA3/OSC2)
- net at X1.3 (X1): now also IC1.9 (RA2/OSC1); no longer IC1.6 (RA2/OSC1)
- net at C8.1: now also IC1.20 (Vcap); no longer IC1.17 (Vcap)
- new net: D2.2 (A), R4.2
- no-connect marks 10 -> 9
Other:
- moved on the sheet: C1, C8, IC1, R5, R6, X1
