File: Boards/AnalogInputV2-0/Analog-Input-Card.sch (KiCad schematic (older format))
At the start: 60 parts, among them IC1 PIC32MM0064GPM028, P1 AquaPicBus, P2 Inputs, P3 Earth, P4 Power, P5 ICSP, Q1 AO3407A, Q2 NX7002AK, Q3 NX7002AK, Q4 NX7002AK, U1 ST485EC, U2 MCP3428, U3 AP2114H, X1 8MHz

Commit message: refactored Digital Input to PIC32
Parts:
- P2: value Inputs -> 1x16 2.54; symbol CONN_01X16 -> Conn_01x16
- P3: value Earth -> 1x2 2.54; symbol CONN_01X02 -> Conn_01x02
- P4: value Power -> 1x2 2.54; symbol CONN_01X02 -> Conn_01x02
Changed lines of the file:
@@
 EESchema Schematic File Version 2
-LIBS:Analog-Input-Card-rescue
 LIBS:power
 LIBS:device
@@
 APB Connectors
 $Comp
-L CONN_01X02 P4
+L Conn_01x02 P4
 U 1 1 558FFC76
-P 9300 5550
-F 0 "P4" H 9300 5700 50  0000 C CNN
-F 1 "Power" V 9400 5550 50  0000 C CNN
-F 2 "MyFootPrints:Screw_Header_1x2" H 9300 5550 60  0001 C CNN
-F 3 "" H 9300 5550 60  0000 C CNN
-	1    9300 5550
+P 9350 5500
+F 0 "P4" H 9350 5600 50  0000 C CNN
+F 1 "1x2 2.54" V 9450 5500 50  0001 C CNN
+F 2 "MyFootPrints:Screw_Header_1x2" H 9350 5500 60  0001 C CNN
+F 3 "" H 9350 5500 60  0000 C CNN
+	1    9350 5500
 	-1   0    0    -1
 $EndComp
@@
 $EndComp
 $Comp
-L CONN_01X16 P2
+L Conn_01x16 P2
 U 1 1 5601E606
-P 10800 1850
-F 0 "P2" H 10800 2700 50  0000 C CNN
-F 1 "Inputs" V 10900 1850 50  0000 C CNN
-F 2 "MyFootPrints:Screw_Header_1x16" H 10800 1850 60  0001 C CNN
-F 3 "" H 10800 1850 60  0000 C CNN
-	1    10800 1850
-	1    0    0    -1
-$EndComp
-$Comp
-L CONN_01X02 P3
+P 10800 1800
+F 0 "P2" H 10800 2600 50  0000 C CNN
+F 1 "1x16 2.54" V 10900 1800 50  0001 C CNN
+F 2 "MyFootPrints:Screw_Header_1x16" H 10800 1800 60  0001 C CNN
+F 3 "" H 10800 1800 60  0000 C CNN
+	1    10800 1800
+	1    0    0    -1
+$EndComp
+$Comp
+L Conn_01x02 P3
 U 1 1 5601FC6C
-P 10800 2950
-F 0 "P3" H 10800 3100 50  0000 C CNN
-F 1 "Earth" V 10900 2950 50  0000 C CNN
-F 2 "MyFootPrints:Screw_Header_1x2" H 10800 2950 60  0001 C CNN
-F 3 "" H 10800 2950 60  0000 C CNN
-	1    10800 2950
+P 10800 2900
+F 0 "P3" H 10800 3000 50  0000 C CNN
+F 1 "1x2 2.54" V 10900 2900 50  0001 C CNN
+F 2 "MyFootPrints:Screw_Header_1x2" H 10800 2900 60  0001 C CNN
+F 3 "" H 10800 2900 60  0000 C CNN
+	1    10800 2900
 	1    0    0    -1
 $EndComp
@@
 L +5V #PWR013
 U 1 1 5A0A0CFE
-P 10200 5400
-F 0 "#PWR013" H 10200 5490 20  0001 C CNN
-F 1 "+5V" H 10200 5490 30  0000 C CNN
-F 2 "~" H 10200 5400 60  0000 C CNN
-F 3 "~" H 10200 5400 60  0000 C CNN
-	1    10200 5400
+P 10150 5450
+F 0 "#PWR013" H 10150 5540 20  0001 C CNN
+F 1 "+5V" H 10150 5540 30  0000 C CNN
+F 2 "~" H 10150 5450 60  0000 C CNN
+F 3 "~" H 10150 5450 60  0000 C CNN
+	1    10150 5450
 	1    0    0    -1
 $EndComp
@@
 L GND #PWR014
 U 1 1 558FD6A3
-P 9600 5700
-F 0 "#PWR014" H 9600 5700 30  0001 C CNN
-F 1 "GND" H 9600 5630 30  0001 C CNN
-F 2 "~" H 9600 5700 60  0000 C CNN
-F 3 "~" H 9600 5700 60  0000 C CNN
-	1    9600 5700
+P 9650 5700
+F 0 "#PWR014" H 9650 5700 30  0001 C CNN
+F 1 "GND" H 9650 5630 30  0001 C CNN
+F 2 "~" H 9650 5700 60  0000 C CNN
+F 3 "~" H 9650 5700 60  0000 C CNN
+	1    9650 5700
 	1    0    0    -1
 $EndComp
@@
 	1300 2700 1700 2700
 Wire Wire Line
-	1600 900  1600 1100
+	1600 900  1600 1000
+Wire Wire Line
+	1600 1000 1600 1100
 Wire Wire Line
 	1600 3000 1700 3000
@@
 	1200 6900 1400 6900
 Wire Wire Line
-	2900 2300 3300 2300
+	2900 2300 3000 2300
+Wire Wire Line
+	3000 2300 3300 2300
 Wire Wire Line
 	1200 6350 1400 6350
@@
 	4100 6900 3900 6900
 Wire Wire Line
-	9500 5600 9600 5600
+	9550 5600 9650 5600
 Wire Wire Line
 	3900 6500 3800 6500
@@
 	3000 7600 4300 7600
 Wire Wire Line
-	9600 5600 9600 5700
+	9650 5600 9650 5700
 Wire Wire Line
 	9800 2400 10600 2400
@@
 	1600 1000 1700 1000
 Wire Wire Line
-	1600 2900 1600 3100
-Wire Wire Line
-	10200 1000 10200 2300
+	1600 2900 1600 3000
+Wire Wire Line
+	1600 3000 1600 3100
+Wire Wire Line
+	10200 1000 10200 1100
+Wire Wire Line
+	10200 1100 10200 1500
+Wire Wire Line
+	10200 1500 10200 1900
+Wire Wire Line
+	10200 1900 10200 2300
 Wire Wire Line
 	10200 1100 10600 1100
@@
 Connection ~ 10300 2100
 Wire Wire Line
-	10300 1300 10300 2700
+	10300 1300 10300 1700
+Wire Wire Line
+	10300 1700 10300 2100
+Wire Wire Line
+	10300 2100 10300 2500
+Wire Wire Line
+	10300 2500 10300 2700
 Wire Wire Line
 	10300 2500 10600 2500
 Connection ~ 10300 2500
 Wire Wire Line
-	10500 1400 10500 3000
+	10500 1400 10500 1800
+Wire Wire Line
+	10500 1800 10500 2200
+Wire Wire Line
+	10500 2200 10500 2600
+Wire Wire Line
+	10500 2600 10500 2900
+Wire Wire Line
+	10500 2900 10500 3000
 Wire Wire Line
 	10500 2600 10600 2600
@@
 	5900 1300 6000 1300
 Wire Wire Line
-	6000 1300 6000 2000
+	6000 1300 6000 1500
+Wire Wire Line
+	6000 1500 6000 1700
+Wire Wire Line
+	6000 1700 6000 1900
+Wire Wire Line
+	6000 1900 6000 2000
 Wire Wire Line
 	5900 1900 6000 1900
@@
 	8000 1500 8000 1600
 Wire Wire Line
-	6900 1500 8100 1500
-Wire Wire Line
-	8400 1500 8500 1500
+	6900 1500 7200 1500
+Wire Wire Line
+	7200 1500 7650 1500
+Wire Wire Line
+	7650 1500 8000 1500
+Wire Wire Line
+	8000 1500 8100 1500
+Wire Wire Line
+	8400 1500 8450 1500
+Wire Wire Line
+	8450 1500 8500 1500
 Wire Wire Line
 	8000 2300 8000 2400
 Wire Wire Line
-	6900 2300 8100 2300
-Wire Wire Line
-	8400 2300 8500 2300
+	6900 2300 7200 2300
+Wire Wire Line
+	7200 2300 7600 2300
+Wire Wire Line
+	7600 2300 8000 2300
+Wire Wire Line
+	8000 2300 8100 2300
+Wire Wire Line
+	8400 2300 8450 2300
+Wire Wire Line
+	8450 2300 8500 2300
 Wire Notes Line
 	2600 7600 2600 5900
@@
 	4800 1400 5100 1400
 Wire Wire Line
-	5000 1600 5000 1800
+	5000 1600 5000 1700
+Wire Wire Line
+	5000 1700 5000 1800
 Wire Wire Line
 	5000 1600 5100 1600
@@
 	8900 1600 8900 1500
 Wire Wire Line
-	8800 1500 9300 1500
+	8800 1500 8900 1500
+Wire Wire Line
+	8900 1500 9300 1500
 Connection ~ 7650 1500
 Wire Wire Line
@@
 	8900 2400 8900 2300
 Wire Wire Line
-	8800 2300 9300 2300
+	8800 2300 8900 2300
+Wire Wire Line
+	8900 2300 9300 2300
 Connection ~ 8900 2300
 Wire Wire Line
 	8000 3100 8000 3200
 Wire Wire Line
-	6900 3100 8100 3100
-Wire Wire Line
-	8400 3100 8500 3100
+	6900 3100 7200 3100
+Wire Wire Line
+	7200 3100 7600 3100
+Wire Wire Line
+	7600 3100 8000 3100
+Wire Wire Line
+	8000 3100 8100 3100
+Wire Wire Line
+	8400 3100 8450 3100
+Wire Wire Line
+	8450 3100 8500 3100
 Connection ~ 7600 3100
 Wire Wire Line
@@
 	8900 3200 8900 3100
 Wire Wire Line
-	8800 3100 9300 3100
+	8800 3100 8900 3100
+Wire Wire Line
+	8900 3100 9300 3100
 Connection ~ 8900 3100
 Wire Wire Line
 	8000 3900 8000 4000
 Wire Wire Line
-	6900 3900 8100 3900
-Wire Wire Line
-	8400 3900 8500 3900
+	6900 3900 7200 3900
+Wire Wire Line
+	7200 3900 7600 3900
+Wire Wire Line
+	7600 3900 8000 3900
+Wire Wire Line
+	8000 3900 8100 3900
+Wire Wire Line
+	8400 3900 8450 3900
+Wire Wire Line
+	8450 3900 8500 3900
 Connection ~ 7600 3900
 Wire Wire Line
@@
 	8900 4000 8900 3900
 Wire Wire Line
-	8800 3900 9300 3900
+	8800 3900 8900 3900
+Wire Wire Line
+	8900 3900 9300 3900
 Connection ~ 8900 3900
 Wire Notes Line
@@
 	10500 2900 10600 2900
 Wire Wire Line
-	10100 5500 10200 5500
-Wire Wire Line
-	10200 5500 10200 5400
+	10100 5500 10150 5500
+Wire Wire Line
+	10150 5500 10150 5450
 Wire Wire Line
 	3900 6800 4100 6800
@@
 Connection ~ 3000 2300
 Wire Wire Line
-	2500 5200 3000 5200
+	2500 5200 2900 5200
+Wire Wire Line
+	2900 5200 3000 5200
 Connection ~ 2900 5200
 Wire Wire Line
-	1900 4400 1900 4600
-Wire Wire Line
-	1400 4900 1600 4900
+	1900 4400 1900 4500
+Wire Wire Line
+	1900 4500 1900 4600
+Wire Wire Line
+	1400 4900 1500 4900
+Wire Wire Line
+	1500 4900 1600 4900
 Wire Wire Line
 	1500 4900 1500 5000
@@
 	3500 4800 3500 4900
 Wire Wire Line
-	2900 4800 2900 4900
+	2900 4800 2900 4850
+Wire Wire Line
+	2900 4850 2900 4900
 Wire Wire Line
 	2900 4850 3100 4850
@@
 Connection ~ 2900 4850
 Wire Wire Line
-	3400 5200 3800 5200
+	3400 5200 3500 5200
+Wire Wire Line
+	3500 5200 3800 5200
 Connection ~ 3500 5200
 $Comp
@@
 $EndComp
 Wire Wire Line
-	2500 4400 3000 4400
+	2500 4400 2900 4400
+Wire Wire Line
+	2900 4400 3000 4400
 Connection ~ 2900 4400
 Wire Wire Line
 	3500 4000 3500 4100
 Wire Wire Line
-	2900 4000 2900 4100
+	2900 4000 2900 4050
+Wire Wire Line
+	2900 4050 2900 4100
 Wire Wire Line
 	2900 4050 3100 4050
@@
 Connection ~ 2900 4050
 Wire Wire Line
-	3400 4400 3800 4400
+	3400 4400 3500 4400
+Wire Wire Line
+	3500 4400 3800 4400
 Connection ~ 3500 4400
 $Comp
@@
 	5000 6450 5000 6500
 Wire Wire Line
-	5000 6500 5800 6500
-Wire Wire Line
-	5400 6450 5400 6550
+	5000 6500 5400 6500
+Wire Wire Line
+	5400 6500 5800 6500
+Wire Wire Line
+	5400 6450 5400 6500
+Wire Wire Line
+	5400 6500 5400 6550
 Wire Wire Line
 	5800 6500 5800 6450
@@
 $EndComp
 Wire Wire Line
-	9700 5500 9500 5500
+	9700 5500 9550 5500
 Wire Wire Line
 	3500 3000 3500 2950
@@
 	1150 1200 1150 1250
 Wire Wire Line
-	1150 1250 1350 1250
+	1150 1250 1250 1250
+Wire Wire Line
+	1250 1250 1350 1250
 Wire Wire Line
 	1350 1250 1350 1200
@@
 	1150 1000 1150 950
 Wire Wire Line
-	1150 950  1350 950
+	1150 950  1250 950
+Wire Wire Line
+	1250 950  1350 950
 Wire Wire Line
 	1350 950  1350 1000
