File: Boards/AnalogInputV2-0/Analog-Input-Card.sch (KiCad schematic (older format))
At the start: 60 parts, among them IC1 PIC32MM0064GPM028, P1 AquaPicBus, P2 1x16 2.54, P3 1x2 2.54, P4 1x2 2.54, P5 ICSP, Q1 AO3407A, Q2 NX7002AK, Q3 NX7002AK, Q4 NX7002AK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

Commit message: must have made changes to some schematics
Connections:
- net Input1: now also RV1.1; no longer RV1.2
- net Input2: now also RV2.1; no longer RV2.2
- net Input3: now also RV3.1; no longer RV3.2
- net Input4: now also RV4.1; no longer RV4.2
- net at R7.1, RV1.3: now also RV1.2
- net at R9.1, RV2.3: now also RV2.2
- net at R11.1, RV3.3: now also RV3.2
- net at R13.1, RV4.3: now also RV4.2
Other:
- moved on the sheet: RV1, RV2, RV3, RV4
Changed lines of the file:
@@
 U 1 1 59F90BCA
 P 8650 1500
-F 0 "RV1" V 8550 1500 50  0000 C CNN
-F 1 "10K" V 8650 1500 50  0000 C CNN
+F 0 "RV1" H 8650 1400 50  0000 C CNN
+F 1 "10K" H 8650 1500 50  0000 C CNN
 F 2 "MyFootPrints:POTENTIAMETER_SMD" H 8650 1500 50  0001 C CNN
 F 3 "" H 8650 1500 50  0001 C CNN
 	1    8650 1500
-	0    1    1    0
+	-1   0    0    1
 $EndComp
 Text Label 6900 1500 0    60   ~ 0
@@
 U 1 1 59F921A7
 P 8650 2300
-F 0 "RV2" V 8550 2300 50  0000 C CNN
-F 1 "10K" V 8650 2300 50  0000 C CNN
+F 0 "RV2" H 8650 2200 50  0000 C CNN
+F 1 "10K" H 8650 2300 50  0000 C CNN
 F 2 "MyFootPrints:POTENTIAMETER_SMD" H 8650 2300 50  0001 C CNN
 F 3 "" H 8650 2300 50  0001 C CNN
 	1    8650 2300
-	0    1    1    0
+	-1   0    0    1
 $EndComp
 Text Label 9300 3100 2    60   ~ 0
@@
 U 1 1 59F92318
 P 8650 3100
-F 0 "RV3" V 8550 3100 50  0000 C CNN
-F 1 "10K" V 8650 3100 50  0000 C CNN
+F 0 "RV3" H 8650 3000 50  0000 C CNN
+F 1 "10K" H 8650 3100 50  0000 C CNN
 F 2 "MyFootPrints:POTENTIAMETER_SMD" H 8650 3100 50  0001 C CNN
 F 3 "" H 8650 3100 50  0001 C CNN
 	1    8650 3100
-	0    1    1    0
+	-1   0    0    1
 $EndComp
 Text Label 6900 3100 0    60   ~ 0
@@
 U 1 1 59F930F5
 P 8650 3900
-F 0 "RV4" V 8550 3900 50  0000 C CNN
-F 1 "10K" V 8650 3900 50  0000 C CNN
+F 0 "RV4" H 8650 3800 50  0000 C CNN
+F 1 "10K" H 8650 3900 50  0000 C CNN
 F 2 "MyFootPrints:POTENTIAMETER_SMD" H 8650 3900 50  0001 C CNN
 F 3 "" H 8650 3900 50  0001 C CNN
 	1    8650 3900
-	0    1    1    0
+	-1   0    0    1
 $EndComp
 Text Label 6900 3900 0    60   ~ 0

Commit message: updated analog input to kicad 5
Parts:
- D1: symbol TRI-LED -> GoodtimeDev:TRI-LED
- IC1: symbol PIC32MM0064GPM028_SSOP -> GoodtimeDev:PIC32MM0064GPM028_SSOP
- P1: symbol USB1.0_Stacked -> GoodtimeDev:USB1.0_Stacked
- Q1: symbol MOSFET_P_SMALL -> GoodtimeDev:MOSFET_P_SMALL
- Q2, Q3, Q4: symbol MOSFET_N_SMALL -> GoodtimeDev:MOSFET_N_SMALL
- U1: symbol SN75176B -> GoodtimeDev:SN75176B
- X1: symbol RESONATOR -> GoodtimeDev:RESONATOR
