File: Boards/AnalogOutputV2-0/Analog-Output-Card.sch (KiCad schematic (older format))
At the start: 74 parts, among them IC1 PIC32MM0064GPM028, P3 Power, P4 Dimming Outputs, Q1 AO3407A, Q2 AO3407A, U1 LM358, U2 LM358, U3 ST485EC, U4 DG469, U5 DG469, U6 DG469, U7 DG469

Commit message: fixed pinout on analog input card
Parts:
- removed Power: 1x2 2.54, MyFootPrints:Screw_Header_1x2, symbol Conn_01x02
- removed Q?: AO3407A, TO_SOT_Packages_SMD:SOT-23, symbol MOSFET_P_SMALL
- removed R? (x2): 4K99, Resistors_SMD:R_0805, symbol R
- added Q? (x4): NX7002AK, TO_SOT_Packages_SMD:SOT-23, symbol MOSFET_N_SMALL
- added R? (x8): 4K99, Resistors_SMD:R_0805, symbol R
- IC1: footprint Housings_DFN_QFN:QFN-28-1EP_6x6mm_Pitch0.65mm -> Housings_SSOP:SSOP-28_5.3x10.2mm_Pitch0.65mm; symbol PIC32MM0064GPM028_QFN -> PIC32MM0064GPM028_SSOP
- U1: symbol LM358_SMALL -> LM358
Connections:
- net labels added: A1, A2, A4, OUT1, OUT2, OUT4, PWM1_LV, PWM2_LV, PWM3_LV, PWM4_LV
- net labels removed: A_OUT1, A_OUT2, A_OUT4, D_OUT1, D_OUT2, D_OUT3, D_OUT4, En_pH, En_pH/ORP, SCL, SDA
- wire segments 220 -> 219
- no-connect marks 8 -> 3
Other:
- moved on the sheet: C1, C11, C12, C13, C14, C15, C16, C17, C18, C2, C3, C5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

Commit message: working on Analog Output card
Parts:
- C15, C16, C17, C18: symbol C-RESCUE-Analog-Output-Card -> C
- D2, D3: footprint LEDs:LED-0805 -> LEDs:LED_0805
- P1: renamed from P4; value Dimming Outputs -> 8x1 2.54; footprint A_MyFootPrints:Screw_Header_1x8 -> MyFootPrints:Screw_Header_1x8
- P3: value Power -> 4x1 2.54
- Q1, Q2: footprint Housings_SOT-23_SOT-143_TSOT-6:SOT-23 -> TO_SOT_Packages_SMD:SOT-23
- U4, U5, U6, U7: footprint A_MyFootPrints:TSSOP-6_SC-70-6 -> Housings_SSOP:TSSOP-8_3x3mm_Pitch0.65mm; symbol TS5A4624 -> DG469
- gave numbers to parts that had none: 28
- renumbered AquaPicBus to P2, ICSP to P4
Connections:
- net +12V: now also U4.4 (V+), U5.4 (V+), U6.4 (V+), U7.4 (V+); no longer U4.2 (Vcc), U5.2 (Vcc), U6.2 (Vcc), U7.2 (Vcc)
- net A1: now also U4.2 (NC); no longer U4.4 (NC)
- net A2: now also U6.2 (NC); no longer U6.4 (NC)
- net A3: now also U5.2 (NC); no longer U5.4 (NC)
- net A4: now also U7.2 (NC); no longer U7.4 (NC)
- net GND: now also U4.7 (V-), U5.7 (V-), U6.7 (V-), U7.7 (V-)
- net OUT1: now also U4.1 (COM); no longer U4.5 (COM)
- net OUT2: now also U6.1 (COM)
- net OUT3: now also U5.1 (COM); no longer U5.5 (COM), U6.5 (COM)
- net OUT4: now also U7.1 (COM); no longer U7.5 (COM)
- net PWM1: now also U4.8 (NO); no longer U4.6 (NO)
- net PWM2: now also U6.8 (NO); no longer U6.6 (NO)
- net PWM3: now also U5.8 (NO); no longer U5.6 (NO)
- net PWM4: now also U7.8 (NO); no longer U7.6 (NO)
- net RELAY1: now also U4.6 (IN); no longer U4.1 (IN)
- net RELAY2: now also U6.6 (IN); no longer U6.1 (IN)
- net RELAY3: now also U5.6 (IN); no longer U5.1 (IN)
- net RELAY4: now also U7.6 (IN); no longer U7.1 (IN)
- net at Q1.3 (D): now also P3.1 (Pin_1); no longer P3.3 (Pin_3)
- net at Q2.3 (D): now also P3.3 (Pin_3); no longer P3.1 (Pin_1)
Other:
- note added: "PWM Level Shifting"
- moved on the sheet: C1, C10, C11, C12, C13, C14, C15, C16, C17, C18, C19, C2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

Commit message: worked on Analog Output Cardboard layout finished
Parts:
- renumbered Q6 to Q4, Q4 to Q5, Q7 to Q6, Q5 to Q7, R19 to R17, R17 to R18, R18 to R19, U6 to U5, U5 to U6
Other:
- moved on the sheet: C16, C17
Changed lines of the file:
@@
 L C C17
 U 1 1 538B9E1D
-P 12600 5700
-F 0 "C17" H 12600 5800 40  0000 L CNN
-F 1 "100nF" H 12606 5615 40  0000 L CNN
-F 2 "Capacitors_SMD:C_0805" H 12638 5550 30  0001 C CNN
-F 3 "~" H 12600 5700 60  0000 C CNN
-	1    12600 5700
+P 8800 7000
+F 0 "C17" H 8800 7100 40  0000 L CNN
+F 1 "100nF" H 8806 6915 40  0000 L CNN
+F 2 "Capacitors_SMD:C_0805" H 8838 6850 30  0001 C CNN
+F 3 "~" H 8800 7000 60  0000 C CNN
+	1    8800 7000
 	-1   0    0    -1
 $EndComp
@@
 L C C16
 U 1 1 538B9E41
-P 8800 7000
-F 0 "C16" H 8800 7100 40  0000 L CNN
-F 1 "100nF" H 8806 6915 40  0000 L CNN
-F 2 "Capacitors_SMD:C_0805" H 8838 6850 30  0001 C CNN
-F 3 "~" H 8800 7000 60  0000 C CNN
-	1    8800 7000
+P 12600 5700
+F 0 "C16" H 12600 5800 40  0000 L CNN
+F 1 "100nF" H 12606 5615 40  0000 L CNN
+F 2 "Capacitors_SMD:C_0805" H 12638 5550 30  0001 C CNN
+F 3 "~" H 12600 5700 60  0000 C CNN
+	1    12600 5700
 	1    0    0    -1
 $EndComp
@@
 $EndComp
 $Comp
-L DG469 U5
+L DG469 U6
 U 1 1 53A08A33
 P 9800 7100
-F 0 "U5" H 9950 7400 60  0000 C CNN
+F 0 "U6" H 9950 7400 60  0000 C CNN
 F 1 "DG469" H 9450 6800 60  0000 C CNN
 F 2 "Housings_SSOP:TSSOP-8_3x3mm_Pitch0.65mm" H 9800 7100 60  0001 C CNN
@@
 $EndComp
 $Comp
-L DG469 U6
+L DG469 U5
 U 1 1 53A08A3B
 P 11600 5800
-F 0 "U6" H 11750 6100 60  0000 C CNN
+F 0 "U5" H 11750 6100 60  0000 C CNN
 F 1 "DG469" H 11250 5500 60  0000 C CNN
 F 2 "Housings_SSOP:TSSOP-8_3x3mm_Pitch0.65mm" H 11600 5800 60  0001 C CNN
@@
 $EndComp
 $Comp
-L R R17
+L R R18
 U 1 1 5A1BA366
 P 3750 4700
-F 0 "R17" V 3830 4700 40  0000 C CNN
+F 0 "R18" V 3830 4700 40  0000 C CNN
 F 1 "150R" V 3757 4701 40  0000 C CNN
 F 2 "Resistors_SMD:R_0805" V 3680 4700 30  0001 C CNN
@@
 $EndComp
 $Comp
-L R R18
+L R R19
 U 1 1 5A1BA36D
 P 3750 4950
-F 0 "R18" V 3830 4950 40  0000 C CNN
+F 0 "R19" V 3830 4950 40  0000 C CNN
 F 1 "150R" V 3757 4951 40  0000 C CNN
 F 2 "Resistors_SMD:R_0805" V 3680 4950 30  0001 C CNN
@@
 $EndComp
 $Comp
-L R R19
+L R R17
 U 1 1 5A1BA374
 P 3750 5200
-F 0 "R19" V 3830 5200 40  0000 C CNN
+F 0 "R17" V 3830 5200 40  0000 C CNN
 F 1 "150R" V 3757 5201 40  0000 C CNN
 F 2 "Resistors_SMD:R_0805" V 3680 5200 30  0001 C CNN
@@
 /RTS
 $Comp
-L MOSFET_N_SMALL Q5
+L MOSFET_N_SMALL Q7
 U 1 1 5A1BA42C
 P 2100 8400
-F 0 "Q5" H 2100 8600 60  0000 R CNN
+F 0 "Q7" H 2100 8600 60  0000 R CNN
 F 1 "NX7002AK" V 2350 8550 60  0000 R CNN
 F 2 "TO_SOT_Packages_SMD:SOT-23" H 2100 8400 60  0001 C CNN
@@
 	5150 1600 5800 1600
 $Comp
-L MOSFET_N_SMALL Q6
+L MOSFET_N_SMALL Q4
 U 1 1 5A1E33C7
 P 6050 2400
-F 0 "Q6" V 5950 2500 60  0000 R CNN
+F 0 "Q4" V 5950 2500 60  0000 R CNN
 F 1 "NX7002AK" V 6300 2550 60  0000 R CNN
 F 2 "TO_SOT_Packages_SMD:SOT-23" H 6050 2400 60  0001 C CNN
@@
 	5200 2500 5850 2500
 $Comp
-L MOSFET_N_SMALL Q4
+L MOSFET_N_SMALL Q5
 U 1 1 5A1E35B7
 P 6100 3300
-F 0 "Q4" V 6000 3400 60  0000 R CNN
+F 0 "Q5" V 6000 3400 60  0000 R CNN
 F 1 "NX7002AK" V 6350 3450 60  0000 R CNN
 F 2 "TO_SOT_Packages_SMD:SOT-23" H 6100 3300 60  0001 C CNN
@@
 	5250 3400 5900 3400
 $Comp
-L MOSFET_N_SMALL Q7
+L MOSFET_N_SMALL Q6
 U 1 1 5A1E3F81
 P 6100 4200
-F 0 "Q7" V 6000 4300 60  0000 R CNN
+F 0 "Q6" V 6000 4300 60  0000 R CNN
 F 1 "NX7002AK" V 6350 4350 60  0000 R CNN
 F 2 "TO_SOT_Packages_SMD:SOT-23" H 6100 4200 60  0001 C CNN

Commit message: refactored Digital Input to PIC32
Parts:
- P1: value 8x1 2.54 -> 1x8 2.54; symbol CONN_01X08 -> Conn_01x08
- P4: value 6x1 2.54 Pin Header -> 2x3 1.27 Pin Header; symbol CONN_01X06 -> Conn_01x06
Changed lines of the file:
@@
 $EndComp
 $Comp
-L CONN_01X08 P1
+L Conn_01x08 P1
 U 1 1 557C01FE
-P 7900 5850
-F 0 "P1" H 7900 6300 50  0000 C CNN
-F 1 "8x1 2.54" V 8000 5850 50  0001 C CNN
-F 2 "MyFootPrints:Screw_Header_1x8" H 7900 5850 60  0001 C CNN
-F 3 "" H 7900 5850 60  0000 C CNN
-	1    7900 5850
+P 7900 5800
+F 0 "P1" H 7900 6200 50  0000 C CNN
+F 1 "1x8 2.54" V 8000 5800 50  0001 C CNN
+F 2 "MyFootPrints:Screw_Header_1x8" H 7900 5800 60  0001 C CNN
+F 3 "" H 7900 5800 60  0000 C CNN
+	1    7900 5800
 	1    0    0    -1
 $EndComp
@@
 APB Connectors
 $Comp
-L CONN_01X06 P4
+L Conn_01x06 P4
 U 1 1 5A1BA3BF
-P 1350 5000
-F 0 "P4" H 1350 5350 50  0000 C CNN
-F 1 "6x1 2.54 Pin Header" V 1350 5000 50  0001 C CNN
-F 2 "Pin_Headers:Pin_Header_Straight_1x06_Pitch2.54mm" H 1350 5000 60  0001 C CNN
-F 3 "" H 1350 5000 60  0000 C CNN
-	1    1350 5000
+P 1350 4950
+F 0 "P4" H 1350 5250 50  0000 C CNN
+F 1 "2x3 1.27 Pin Header" V 1350 4950 50  0001 C CNN
+F 2 "Pin_Headers:Pin_Header_Straight_1x06_Pitch2.54mm" H 1350 4950 60  0001 C CNN
+F 3 "" H 1350 4950 60  0000 C CNN
+	1    1350 4950
 	-1   0    0    -1
 $EndComp
