File: Boards/DigitalInputV2-0/Digital-Input-Card.kicad_pcb (KiCad board)
At the start: 2 copper layers, 80 x 72 mm, 44 parts, among them IC1 PIC32MM0064GPM028, P1 1x6 2.54 Pin Header, P2 1x12 2.54, P3 1x2 2.54, P4 1x4 2.54, P5 Stacked USBA, Q1 AO3407A, Q2 NX7002AK, Q3 NX7002AK, Q4 NX7002AK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

Commit message: worked on charlieplexed led circuit design
Parts:
- R1, R2, R3: value 150R -> 20R
Changed lines of the file:
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@@
       (effects (font (size 1 1) (thickness 0.15)))
     )
-    (fp_text value 150R (at 0 1.75 270) (layer F.Fab)
+    (fp_text value 20R (at 0 1.75 270) (layer F.Fab)
       (effects (font (size 1 1) (thickness 0.15)))
     )
@@
       (effects (font (size 1 1) (thickness 0.15)))
     )
-    (fp_text value 150R (at 0 1.75 270) (layer F.Fab)
+    (fp_text value 20R (at 0 1.75 270) (layer F.Fab)
       (effects (font (size 1 1) (thickness 0.15)))
     )
@@
       (effects (font (size 1 1) (thickness 0.15)))
     )
-    (fp_text value 150R (at 0 1.75 270) (layer F.Fab)
+    (fp_text value 20R (at 0 1.75 270) (layer F.Fab)
       (effects (font (size 1 1) (thickness 0.15)))
     )
