File: Boards/DigitalInput/Digital-Input-Card.sch (KiCad schematic (older format))
At the start: 42 parts, among them IC1 PIC32MM0064GPM028, P1 ICSP, P2 Inputs, P3 5Vdc, P4 Input Power, P5 AquaPicBus, Q1 AO3407A, Q2 NX7002AK, Q3 NX7002AK, Q4 NX7002AK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

Commit message: fixed icsp footprint
Parts:
- P1: footprint Pin_Headers:Pin_Header_Straight_1x06_Pitch2.54mm -> Connector_PinHeader_2.54mm:PinHeader_1x06_P2.54mm_Vertical
Changed lines of the file:
@@
 F 0 "P1" H 4350 1650 50  0000 C CNN
 F 1 "ICSP" V 4350 1350 50  0001 C CNN
-F 2 "Pin_Headers:Pin_Header_Straight_1x06_Pitch2.54mm" H 4350 1350 60  0001 C CNN
+F 2 "Connector_PinHeader_2.54mm:PinHeader_1x06_P2.54mm_Vertical" H 4350 1350 60  0001 C CNN
 F 3 "" H 4350 1350 60  0000 C CNN
 F 4 "1x6 2.54 Male Pin Header" H 200 0   50  0001 C CNN "Type"
