File: Boards/AnalogOutput/Analog-Output-Card.sch (KiCad schematic (older format))
At the start: 82 parts, among them IC1 PIC32MM0064GPM028, P1 1x8 2.54, P2 Stacked USBA, P3 4x1 2.54, P4 2x3 1.27 Pin Header, Q1 AO3407A, Q2 AO3407A, Q3 NX7002AK, Q4 NX7002AK, Q5 NX7002AK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

Commit message: analog output bom is not controlled by schematic
Parts:
- C1, C13, C14, C15, C16, C17, C18, C2, C20, C3, C4, C7, C8, C9: Comments (none) -> 0805, 50V, X7R, 10%; Digi-Key Part Number (none) -> 399-1170-1-ND; Manufacturer (none) -> Kemet; Manufacturer Part Number (none) -> C0805C104K5RACTU; Type (none) -> Capacitor
- C10, C19: Comments (none) -> 0805, 10V, X7R, 10%; Digi-Key Part Number (none) -> 1276-2972-1-ND; Manufacturer (none) -> Samsung; Manufacturer Part Number (none) -> CL21B475KPFNNNE; Type (none) -> Capacitor
- C11, C12, C5, C6: Comments (none) -> 0805, 50V, X7R, 10%; Digi-Key Part Number (none) -> 1276-6478-1-ND; Manufacturer (none) -> Samsung; Manufacturer Part Number (none) -> CL21B224KBFNNNG; Type (none) -> Capacitor
- D1: Comments (none) -> 4-PLCC; Digi-Key Part Number (none) -> 492-2173-1-ND; Manufacturer (none) -> Bivar; Manufacturer Part Number (none) -> SMTL4-RGY; Type (none) -> LED (Red, Green, Yellow)
- D2, D3: Comments (none) -> 0805, 2V, 20mA; Digi-Key Part Number (none) -> 475-1278-1-ND; Manufacturer (none) -> Osram; Manufacturer Part Number (none) -> LS R976-NR-1; Type (none) -> LED (Red)
- IC1: Comments (none) -> 28-SSOP 5.3mm; Digi-Key Part Number (none) -> PIC32MM0064GPM028-I/SS-ND; Manufacturer (none) -> Microchip; Manufacturer Part Number (none) -> PIC32MM0064GPM028-I/SS; Type (none) -> Microcontroller
- P1: value 1x8 2.54 -> Outputs; Comments (none) -> -; Digi-Key Part Number (none) -> ED10566-ND; Manufacturer (none) -> ON Shore; Manufacturer Part Number (none) -> OSTVN08A150; Type (none) -> 1x8 2.54 Screw Header
- P2: value Stacked USBA -> AquaPicBus; Comments (none) -> -; Digi-Key Part Number (none) -> 1175-1003-ND; Manufacturer (none) -> CNC Tech; Manufacturer Part Number (none) -> 1001-004-01010; Type (none) -> USB 1.1 Type A
- P3: value 4x1 2.54 -> Power; Comments (none) -> -; Digi-Key Part Number (none) -> ED10563-ND; Manufacturer (none) -> ON Shore; Manufacturer Part Number (none) -> OSTVN04A150; Type (none) -> 1x4 2.54 Screw Header
- P4: value 2x3 1.27 Pin Header -> ICSP; Comments (none) -> -; Digi-Key Part Number (none) -> A105161CT-ND; Manufacturer (none) -> TE; Manufacturer Part Number (none) -> 5-146868-1; Type (none) -> 1x6 2.54 Male Pin Header
- Q1, Q2: Comments (none) -> SOT-23-3; Digi-Key Part Number (none) -> 785-1006-1-ND; Manufacturer (none) -> Alpha Omega; Manufacturer Part Number (none) -> AO3407A; Type (none) -> P-Channel MOSFET
- Q3, Q4, Q5, Q6, Q7, Q8, Q9: Comments (none) -> SOT-23-3; Digi-Key Part Number (none) -> 1727-1289-6-ND; Manufacturer (none) -> Nexperia; Manufacturer Part Number (none) -> NX7002AK,215; Type (none) -> N-Channel MOSFET
- R1, R10, R11, R12, R14, R16, R2, R25, R28, R3, R4, R6, R8, R9: Comments (none) -> 0805, 1/4W, 1%, Thin Film; Digi-Key Part Number (none) -> RNCP0805FTD10K0CT-ND; Manufacturer (none) -> Stackpole; Manufacturer Part Number (none) -> RNCP0805FTD10K0; Type (none) -> Resistor
- R13, R15, R5, R7: Comments (none) -> 0805, 1/4W, 1%, Thin Film; Digi-Key Part Number (none) -> RMCF0805FT100KCT-ND; Manufacturer (none) -> Stackpole; Manufacturer Part Number (none) -> RMCF0805FT100K; Type (none) -> Resistor
- R17, R18, R19, R20: Comments (none) -> 0805, 1/4W, 1%, Thin Film; Digi-Key Part Number (none) -> RNCP0805FTD150RCT-ND; Manufacturer (none) -> Stackpole; Manufacturer Part Number (none) -> RNCP0805FTD150R; Type (none) -> Resistor
- R21, R24: Comments (none) -> 0805, 1/4W, 1%, Thin Film; Digi-Key Part Number (none) -> RNCP0805FTD1K00CT-ND; Manufacturer (none) -> Stackpole; Manufacturer Part Number (none) -> RNCP0805FTD1K00; Type (none) -> Resistor
- R22, R23, R26, R27, R29, R30, R31, R32, R33, R34, R35, R36: Comments (none) -> 0805, 1/4W, 1%, Thin Film; Digi-Key Part Number (none) -> RNCP0805FTD4K99CT-ND; Manufacturer (none) -> Stackpole; Manufacturer Part Number (none) -> RNCP0805FTD4K99; Type (none) -> Resistor
- U1, U2: Comments (none) -> 8-TSSOP 4.4mm; Digi-Key Part Number (none) -> 296-9555-1-ND; Manufacturer (none) -> Texas; Manufacturer Part Number (none) -> LM358PWR; Type (none) -> OpAmp
- U3: Comments (none) -> 8-SOIC 3.9mm; Digi-Key Part Number (none) -> 497-3735-1-ND; Manufacturer (none) -> STMicro; Manufacturer Part Number (none) -> ST485ECDR; Type (none) -> RS485 Transceiver
- U4, U5, U6, U7: Comments (none) -> 8-TSSOP 3mm; Digi-Key Part Number (none) -> DG469EQ-T1-E3CT-ND; Manufacturer (none) -> Vishay; Manufacturer Part Number (none) -> DG469EQ-T1-E3; Type (none) -> SPDT Switch
- U8: Comments (none) -> SOT-223; Digi-Key Part Number (none) -> AP2114HA-2.5TRG1DICT-ND; Manufacturer (none) -> Diodes; Manufacturer Part Number (none) -> AP2114HA-2.5TRG1; Type (none) -> Linear Regulator
- X1: Comments (none) -> 3-SMD, Non-Standard; Digi-Key Part Number (none) -> 490-1195-1-ND; Manufacturer (none) -> Murata; Manufacturer Part Number (none) -> CSTCE8M00G55-R0; Type (none) -> Resonator
