File: Boards/AnalogInput/Analog-Input-Card.sch (KiCad schematic (older format))
At the start: 60 parts, among them IC1 PIC32MM0064GPM028, P1 AquaPicBus, P2 1x16 2.54, P3 1x2 2.54, P4 1x2 2.54, P5 ICSP, Q1 AO3407A, Q2 NX7002AK, Q3 NX7002AK, Q4 NX7002AK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

Commit message: updated analog input to kicad 5
Parts:
- C1, C10, C11, C4, C5, C6, C7, C8, C9: symbol C_Small -> Analog-Input-Card-rescue:C_Small
- C2, C3: symbol C-RESCUE-Analog-Input-Card -> Analog-Input-Card-rescue:C_Small
- D10, D4, D6, D8: symbol D_TVS_ALT -> Analog-Input-Card-rescue:D_TVS_ALT
- D2: symbol LED_ALT -> Analog-Input-Card-rescue:LED_ALT
- D3, D5, D7, D9: symbol D_Zener_ALT -> Analog-Input-Card-rescue:D_Zener_ALT
- P2: symbol Conn_01x16 -> Analog-Input-Card-rescue:Conn_01x16
- P3, P4: symbol Conn_01x02 -> Analog-Input-Card-rescue:Conn_01x02
- P5: symbol CONN_01X06 -> Analog-Input-Card-rescue:CONN_01X06
- R1, R10, R11, R12, R13, R14, R15, R16, R17, R18, R19, R2, R20, R21, R3, R4, R5, R6, R7, R8, R9: symbol R -> Analog-Input-Card-rescue:R
- RV1, RV2, RV3, RV4: symbol POT -> Analog-Input-Card-rescue:POT
- U2: symbol MCP3428 -> Analog-Input-Card-rescue:MCP3428
- U3: symbol AP1117-33 -> Analog-Input-Card-rescue:AP1117-33
Changed lines of the file:
@@
 TX
 $Comp
-L C-RESCUE-Analog-Input-Card C2
+L Analog-Input-Card-rescue:C_Small C2
 U 1 1 558FD6D4
 P 900 6300
@@
 L power:GND #PWR08
 U 1 1 558FD6DB
-P 900 6500
-F 0 "#PWR08" H 900 6500 30  0001 C CNN
-F 1 "GND" H 900 6430 30  0001 C CNN
-F 2 "~" H 900 6500 60  0000 C CNN
-F 3 "~" H 900 6500 60  0000 C CNN
-	1    900  6500
+P 900 6400
+F 0 "#PWR08" H 900 6400 30  0001 C CNN
+F 1 "GND" H 900 6330 30  0001 C CNN
+F 2 "~" H 900 6400 60  0000 C CNN
+F 3 "~" H 900 6400 60  0000 C CNN
+	1    900  6400
 	1    0    0    -1
 $EndComp
@@
 APB Connectors
 $Comp
-L Conn_01x02 P4
+L Analog-Input-Card-rescue:Conn_01x02 P4
 U 1 1 558FFC76
 P 9350 5500
@@
 $EndComp
 $Comp
-L Conn_01x16 P2
+L Analog-Input-Card-rescue:Conn_01x16 P2
 U 1 1 5601E606
 P 10800 1800
@@
 $EndComp
 $Comp
-L Conn_01x02 P3
+L Analog-Input-Card-rescue:Conn_01x02 P3
 U 1 1 5601FC6C
 P 10800 2900
@@
 $EndComp
 $Comp
-L CONN_01X06 P5
+L Analog-Input-Card-rescue:CONN_01X06 P5
 U 1 1 5681CCD0
 P 4950 3200
@@
 $EndComp
 $Comp
-L MCP3428 U2
+L Analog-Input-Card-rescue:MCP3428 U2
 U 1 1 59F7C7E9
 P 5500 1500
@@
 Ch4
 $Comp
-L C-RESCUE-Analog-Input-Card C3
+L Analog-Input-Card-rescue:C_Small C3
 U 1 1 59F802E0
 P 4500 1200
@@
 $EndComp
 $Comp
-L R R7
+L Analog-Input-Card-rescue:R R7
 U 1 1 59F90487
 P 8250 1500
@@
 $EndComp
 $Comp
-L R R8
+L Analog-Input-Card-rescue:R R8
 U 1 1 59F90597
 P 8000 1750
@@
 Ch1
 $Comp
-L POT RV1
+L Analog-Input-Card-rescue:POT RV1
 U 1 1 59F90BCA
 P 8650 1500
@@
 Input2
 $Comp
-L R R9
+L Analog-Input-Card-rescue:R R9
 U 1 1 59F9219B
 P 8250 2300
@@
 $EndComp
 $Comp
-L R R10
+L Analog-Input-Card-rescue:R R10
 U 1 1 59F921A1
 P 8000 2550
@@
 $EndComp
 $Comp
-L POT RV2
+L Analog-Input-Card-rescue:POT RV2
 U 1 1 59F921A7
 P 8650 2300
@@
 Input3
 $Comp
-L R R11
+L Analog-Input-Card-rescue:R R11
 U 1 1 59F9230C
 P 8250 3100
@@
 $EndComp
 $Comp
-L R R12
+L Analog-Input-Card-rescue:R R12
 U 1 1 59F92312
 P 8000 3350
@@
 $EndComp
 $Comp
-L POT RV3
+L Analog-Input-Card-rescue:POT RV3
 U 1 1 59F92318
 P 8650 3100
@@
 Input4
 $Comp
-L R R13
+L Analog-Input-Card-rescue:R R13
 U 1 1 59F930E9
 P 8250 3900
@@
 $EndComp
 $Comp
-L R R14
+L Analog-Input-Card-rescue:R R14
 U 1 1 59F930EF
 P 8000 4150
@@
 $EndComp
 $Comp
-L POT RV4
+L Analog-Input-Card-rescue:POT RV4
 U 1 1 59F930F5
 P 8650 3900
@@
 L power:+5V #PWR012
 U 1 1 59F95AC2
-P 900 6100
-F 0 "#PWR012" H 900 6190 20  0001 C CNN
-F 1 "+5V" H 900 6190 30  0000 C CNN
-F 2 "~" H 900 6100 60  0000 C CNN
-F 3 "~" H 900 6100 60  0000 C CNN
-	1    900  6100
+P 900 6200
+F 0 "#PWR012" H 900 6290 20  0001 C CNN
+F 1 "+5V" H 900 6290 30  0000 C CNN
+F 2 "~" H 900 6200 60  0000 C CNN
+F 3 "~" H 900 6200 60  0000 C CNN
+	1    900  6200
 	1    0    0    -1
 $EndComp
@@
 SCL
 $Comp
-L R R5
+L Analog-Input-Card-rescue:R R5
 U 1 1 59F9BA38
 P 3500 2800
@@
 $EndComp
 $Comp
-L R R6
+L Analog-Input-Card-rescue:R R6
 U 1 1 59F9BC5D
 P 3500 1700
@@
 Input Protection and Voltage Dividers
 $Comp
-L D_TVS_ALT D4
+L Analog-Input-Card-rescue:D_TVS_ALT D4
 U 1 1 5A08195A
 P 8900 1750
@@
 $EndComp
 $Comp
-L D_Zener_ALT D3
+L Analog-Input-Card-rescue:D_Zener_ALT D3
 U 1 1 5A08C32C
 P 7650 1750
@@
 $EndComp
 $Comp
-L C_Small C4
+L Analog-Input-Card-rescue:C_Small C4
 U 1 1 5A08F843
 P 7200 1750
@@
 $EndComp
 $Comp
-L D_Zener_ALT D5
+L Analog-Input-Card-rescue:D_Zener_ALT D5
 U 1 1 5A09261E
 P 7600 2550
@@
 $EndComp
 $Comp
-L C_Small C5
+L Analog-Input-Card-rescue:C_Small C5
 U 1 1 5A092627
 P 7200 2550
@@
 Ch2
 $Comp
-L D_TVS_ALT D6
+L Analog-Input-Card-rescue:D_TVS_ALT D6
 U 1 1 5A0929BA
 P 8900 2550
@@
 $EndComp
 $Comp
-L D_Zener_ALT D7
+L Analog-Input-Card-rescue:D_Zener_ALT D7
 U 1 1 5A092CB1
 P 7600 3350
@@
 $EndComp
 $Comp
-L C_Small C6
+L Analog-Input-Card-rescue:C_Small C6
 U 1 1 5A092CBA
 P 7200 3350
@@
 $EndComp
 $Comp
-L D_TVS_ALT D8
+L Analog-Input-Card-rescue:D_TVS_ALT D8
 U 1 1 5A092CC9
 P 8900 3350
@@
 $EndComp
 $Comp
-L D_Zener_ALT D9
+L Analog-Input-Card-rescue:D_Zener_ALT D9
 U 1 1 5A0938BC
 P 7600 4150
@@
 $EndComp
 $Comp
-L C_Small C7
+L Analog-Input-Card-rescue:C_Small C7
 U 1 1 5A0938C5
 P 7200 4150
@@
 $EndComp
 $Comp
-L D_TVS_ALT D10
+L Analog-Input-Card-rescue:D_TVS_ALT D10
 U 1 1 5A0938D3
 P 8900 4150
@@
 $EndComp
 $Comp
-L C_Small C1
+L Analog-Input-Card-rescue:C_Small C1
 U 1 1 5A0A460A
 P 1350 1100
@@
 $EndComp
 $Comp
-L C_Small C8
+L Analog-Input-Card-rescue:C_Small C8
 U 1 1 5A0A5112
 P 1600 1500
@@
 RX_LV
 $Comp
-L R R17
+L Analog-Input-Card-rescue:R R17
 U 1 1 5A099F8F
 P 2900 5050
@@
 $EndComp
 $Comp
-L R R18
+L Analog-Input-Card-rescue:R R18
 U 1 1 5A099F95
 P 3500 5050
@@
 $EndComp
 $Comp
-L R R19
+L Analog-Input-Card-rescue:R R19
 U 1 1 5A09A531
 P 1250 4900
@@
 $EndComp
 $Comp
-L R R20
+L Analog-Input-Card-rescue:R R20
 U 1 1 5A09A66C
 P 1500 5150
@@
 $EndComp
 $Comp
-L R R21
+L Analog-Input-Card-rescue:R R21
 U 1 1 5A09A792
 P 1900 4250
@@
 L power:GND #PWR038
 U 1 1 5A0A3B87
-P 4500 1400
-F 0 "#PWR038" H 4500 1400 30  0001 C CNN
-F 1 "GND" H 4500 1330 30  0001 C CNN
-F 2 "~" H 4500 1400 60  0000 C CNN
-F 3 "~" H 4500 1400 60  0000 C CNN
-	1    4500 1400
+P 4500 1300
+F 0 "#PWR038" H 4500 1300 30  0001 C CNN
+F 1 "GND" H 4500 1230 30  0001 C CNN
+F 2 "~" H 4500 1300 60  0000 C CNN
+F 3 "~" H 4500 1300 60  0000 C CNN
+	1    4500 1300
 	1    0    0    -1
 $EndComp
@@
 L power:+3.3V #PWR045
 U 1 1 5A0AC36B
-P 4500 1000
-F 0 "#PWR045" H 4500 850 50  0001 C CNN
-F 1 "+3.3V" H 4500 1100 30  0000 C CNN
-F 2 "" H 4500 1000 50  0001 C CNN
-F 3 "" H 4500 1000 50  0001 C CNN
-	1    4500 1000
+P 4500 1100
+F 0 "#PWR045" H 4500 950 50  0001 C CNN
+F 1 "+3.3V" H 4500 1200 30  0000 C CNN
+F 2 "" H 4500 1100 50  0001 C CNN
+F 3 "" H 4500 1100 50  0001 C CNN
+	1    4500 1100
 	1    0    0    -1
 $EndComp
@@
 $EndComp
 $Comp
-L R R15
+L Analog-Input-Card-rescue:R R15
 U 1 1 5A0D44F0
 P 2900 4250
@@
 $EndComp
 $Comp
-L R R16
+L Analog-Input-Card-rescue:R R16
 U 1 1 5A0D44F6
 P 3500 4250
@@
 	700  5600 3900 5600
 $Comp
-L AP1117-33 U3
+L Analog-Input-Card-rescue:AP1117-33 U3
 U 1 1 5A0E5871
 P 5400 6150
@@
 	5000 6150 5100 6150
 $Comp
-L C_Small C10
+L Analog-Input-Card-rescue:C_Small C10
 U 1 1 5A0E619E
 P 5800 6350
@@
 	5800 6150 5700 6150
 $Comp
-L C_Small C9
+L Analog-Input-Card-rescue:C_Small C9
 U 1 1 5A0E6464
 P 5000 6350
@@
 	1650 1800 1700 1800
 $Comp
-L C_Small C11
+L Analog-Input-Card-rescue:C_Small C11
 U 1 1 5A20C8F1
 P 1150 1100
@@
 $EndComp
 $Comp
-L R R1
+L Analog-Input-Card-rescue:R R1
 U 1 1 5A20DA87
 P 5550 4400
@@
 $EndComp
 $Comp
-L R R2
+L Analog-Input-Card-rescue:R R2
 U 1 1 5A20DA8E
 P 5550 4650
@@
 $EndComp
 $Comp
-L R R3
+L Analog-Input-Card-rescue:R R3
 U 1 1 5A20DA95
 P 5550 4900
@@
 $EndComp
 $Comp
-L LED_ALT D2
+L Analog-Input-Card-rescue:LED_ALT D2
 U 1 1 5A20DAA6
 P 7800 5600
@@
 $EndComp
 $Comp
-L R R4
+L Analog-Input-Card-rescue:R R4
 U 1 1 5A20DAAD
 P 7400 5600

Commit message: analog input bom is now controlled by schematic
Parts:
- C1, C11, C2, C3, C4, C5, C6, C7, C8: Comments (none) -> 0805, 50V, X7R, 10%; Digi-Key Part Number (none) -> 445-7534-1-ND; Manufacturer (none) -> TDK; Manufacturer Part Number (none) -> C2012X7R1H104K085AA; Type (none) -> Capacitor
- C10, C9: Comments (none) -> 0805, 10V, X7R, 10%; Digi-Key Part Number (none) -> 1276-2972-1-ND; Manufacturer (none) -> Samsung; Manufacturer Part Number (none) -> CL21B475KPFNNNE; Type (none) -> Capacitor
- D1: Comments (none) -> 4-PLCC; Digi-Key Part Number (none) -> 492-2173-1-ND; Manufacturer (none) -> Bivar; Manufacturer Part Number (none) -> SMTL4-RGY; Type (none) -> LED (Red, Green, Yellow)
- D10, D4, D6, D8: Comments (none) -> SMB, 30V; Digi-Key Part Number (none) -> SMBJ30D-M3/HGICT-ND; Manufacturer (none) -> Vishay; Manufacturer Part Number (none) -> SMBJ30D-M3/H; Type (none) -> TVS
- D2: Comments (none) -> 0805, 2V, 20mA; Digi-Key Part Number (none) -> 475-1278-1-ND; Manufacturer (none) -> Osram; Manufacturer Part Number (none) -> LS R976-NR-1; Type (none) -> LED (Red)
- D3, D5, D7, D9: Comments (none) -> SOT-23-3, 3.3V; Digi-Key Part Number (none) -> BZX84C3V3LT1GOSCT-ND; Manufacturer (none) -> On Semi; Manufacturer Part Number (none) -> BZX84C3V3LT1G; Type (none) -> Zener
- IC1: Comments (none) -> 28-SSOP 5.3mm; Digi-Key Part Number (none) -> PIC32MM0064GPM028-I/SS-ND; Manufacturer (none) -> Microchip; Manufacturer Part Number (none) -> PIC32MM0064GPM028-I/SS; Type (none) -> Microcontroller
- P1: Comments (none) -> 1175-1003-ND; Digi-Key Part Number (none) -> 1175-1003-ND; Manufacturer (none) -> CNC Tech; Manufacturer Part Number (none) -> 1001-004-01010; Type (none) -> USB 1.1 Type A
- P2: value 1x16 2.54 -> Inputs; Comments (none) -> x2; Digi-Key Part Number (none) -> ED10566-ND; Manufacturer (none) -> On Shore; Manufacturer Part Number (none) -> OSTVN08A150; Type (none) -> 1x8 2.54 Screw Header
- P3: value 1x2 2.54 -> Earth; Comments (none) -> -; Digi-Key Part Number (none) -> ED10561-ND; Manufacturer (none) -> On Shore; Manufacturer Part Number (none) -> OSTVN02A150; Type (none) -> 1x2 2.54 Screw Header
- P4: value 1x2 2.54 -> Power; Comments (none) -> -; Digi-Key Part Number (none) -> ED10561-ND; Manufacturer (none) -> On Shore; Manufacturer Part Number (none) -> OSTVN02A150; Type (none) -> 1x2 2.54 Screw Header
- P5: Comments (none) -> -; Digi-Key Part Number (none) -> A105161CT-ND; Manufacturer (none) -> TE; Manufacturer Part Number (none) -> 5-146868-1; Type (none) -> 1x6 Male Pin Header
- Q1: Comments (none) -> SOT-23-3; Digi-Key Part Number (none) -> 785-1006-1-ND; Manufacturer (none) -> Alpha Omega; Manufacturer Part Number (none) -> AO3407A; Type (none) -> P-Channel MOSFET
- Q2, Q3, Q4: Comments (none) -> SOT-23-3; Digi-Key Part Number (none) -> 1727-1289-6-ND; Manufacturer (none) -> Nexperia; Manufacturer Part Number (none) -> NX7002AK,215; Type (none) -> N-Channel MOSFET
- R1, R2, R3, R4: Comments (none) -> 0805, 1/4W, 1%, Thin Film; Digi-Key Part Number (none) -> RNCP0805FTD150RCT-ND; Manufacturer (none) -> Stackpole; Manufacturer Part Number (none) -> RNCP0805FTD150R; Type (none) -> Resistor
- R10, R12, R14, R8: Comment 0805, 1/4W, 1%, Thin Film -> (none); Comments (none) -> 0805, 1/4W, 1%, Thin Film; Digi-Key Part Number (none) -> RNCP0805FTD10K0CT-ND; Manufacturer (none) -> Stackpole; Manufacturer Part Number (none) -> RNCP0805FTD10K0; Type (none) -> Resistor
- R11, R13, R7, R9: Comment 0805, 1/4W, 1%, Thin Film -> (none); Comments (none) -> 0805, 1/4W, 1%, Thin Film; Digi-Key Part Number (none) -> RNCP0805FTD4K99CT-ND; Manufacturer (none) -> Stackpole; Manufacturer Part Number (none) -> RNCP0805FTD4K99; Type (none) -> Resistor
- R15, R16, R17, R18, R5, R6: Comments (none) -> 0805, 1/4W, 1%, Thin Film; Digi-Key Part Number (none) -> RNCP0805FTD4K99CT-ND; Manufacturer (none) -> Stackpole; Manufacturer Part Number (none) -> RNCP0805FTD4K99; Type (none) -> Resistor
- R19: Comments (none) -> 0805, 1/4W, 1%, Thin Film; Digi-Key Part Number (none) -> RNCP0805FTD1K00CT-ND; Manufacturer (none) -> Stackpole; Manufacturer Part Number (none) -> RNCP0805FTD1K00; Type (none) -> Resistor
- R20, R21: Comments (none) -> 0805, 1/4W, 1%, Thin Film; Digi-Key Part Number (none) -> RNCP0805FTD10K0CT-ND; Manufacturer (none) -> Stackpole; Manufacturer Part Number (none) -> RNCP0805FTD10K0; Type (none) -> Resistor
- RV1, RV2, RV3, RV4: Comments (none) -> J Lead, 12T; Digi-Key Part Number (none) -> 987-1155-ND; Manufacturer (none) -> TT; Manufacturer Part Number (none) -> 84WR10KLF; Type (none) -> Potentiomenter
- U1: Comments (none) -> 8-SOIC 3.9mm; Digi-Key Part Number (none) -> 497-3735-1-ND; Manufacturer (none) -> STMicro; Manufacturer Part Number (none) -> ST485ECDR; Type (none) -> RS485 Transceiver
- U2: Comments (none) -> 14-TSSOP 4.4mm; Digi-Key Part Number (none) -> MCP3428-E/ST-ND; Manufacturer (none) -> Microchip; Manufacturer Part Number (none) -> MCP3428-E/ST; Type (none) -> DeltaSigma ADC
- U3: Comments (none) -> SOT-223; Digi-Key Part Number (none) -> AP2114HA-2.5TRG1DICT-ND; Manufacturer (none) -> Diodes; Manufacturer Part Number (none) -> AP2114HA-2.5TRG1; Type (none) -> Linear Regulator
- X1: Comments (none) -> 3-SMD, Non-Standard; Digi-Key Part Number (none) -> 490-1195-1-ND; Manufacturer (none) -> Murata; Manufacturer Part Number (none) -> CSTCE8M00G55-R0; Type (none) -> Resonator
